Commit message: Finalizing professional environment setup with README and optimized configuration

File: src/dynamic_obstacle_pkg/resource/super_car.urdf (robot description, URDF)
Before this commit: robot super_car, 8 links, 7 joints
Links:
- removed link fl_wheel_visual
- removed link fr_wheel_visual
- removed link rl_wheel_visual
- removed link rr_wheel_visual
- added link fl_wheel; visual cylinder length=0.3 radius=0.4
- added link fr_wheel; visual cylinder length=0.3 radius=0.4
- added link rl_wheel; visual cylinder length=0.3 radius=0.4
- added link rr_wheel; visual cylinder length=0.3 radius=0.4
Joints:
- joint fl_j: child fl_wheel_visual -> fl_wheel; origin xyz=0 0 0 rpy=1.5707 0 0 -> xyz=0 0 0 rpy=0 0 0
- joint fr_j: child fr_wheel_visual -> fr_wheel; origin xyz=0 0 0 rpy=1.5707 0 0 -> xyz=0 0 0 rpy=0 0 0
- joint rl_j: child rl_wheel_visual -> rl_wheel; origin xyz=-1.5 0.8 0 rpy=1.5707 0 0 -> xyz=-1.5 0.8 0 rpy=0 0 0
- joint rr_j: child rr_wheel_visual -> rr_wheel; origin xyz=-1.5 -0.8 0 rpy=1.5707 0 0 -> xyz=-1.5 -0.8 0 rpy=0 0 0

Commit message: Corrected car tire positions and visuals for professional alignment in RViz and Gazebo

File: src/dynamic_obstacle_pkg/resource/super_car.urdf (robot description, URDF)
Before this commit: robot super_car, 8 links, 7 joints
Links:
- link base_link: geometry collision box size=4.5 2.2 1.2; visual mesh filename=https://fuel.gazebosim.org/1.0/openrobotics/models/suv/4/me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 scale=0.06 0.06 0.06
- link fl_wheel: geometry visual cylinder length=0.3 radius=0.38
- link fr_wheel: geometry visual cylinder length=0.3 radius=0.38
- link lidar_link: geometry visual cylinder length=0.1 radius=0.1
Joints:
- joint fl_steer_j: origin xyz=1.5 0.8 0 rpy=0 0 0 -> xyz=1.45 0.85 -0.1 rpy=0 0 0
- joint fr_steer_j: origin xyz=1.5 -0.8 0 rpy=0 0 0 -> xyz=1.45 -0.85 -0.1 rpy=0 0 0
- joint lidar_joint: origin xyz=0 0 1.5 rpy=0 0 0 -> xyz=0 0 1.2 rpy=0 0 0
- joint rl_j: origin xyz=-1.5 0.8 0 rpy=0 0 0 -> xyz=-1.45 0.85 -0.1 rpy=0 0 0
- joint rr_j: origin xyz=-1.5 -0.8 0 rpy=0 0 0 -> xyz=-1.45 -0.85 -0.1 rpy=0 0 0
