Commit message: fixes

File: src/dynamic_obstacle_pkg/urdf/super_car.urdf.xacro (robot description, xacro)
@@ -1,142 +1,51 @@
 <?xml version="1.0"?>
 <robot xmlns:xacro="http://www.ros.org/wiki/xacro" name="super_car">
-  <!--
-    super_car.urdf.xacro
-    Ackermann 4.5m x 2m, 0.4m wheel radius, LiDAR at z=1.5m
-    This URDF defines kinematics + sensor frames for:
-      - robot_state_publisher (TF tree)
-      - Nav2 costmap transforms
-      - SLAM scan matching
-    Motion is handled by Gazebo AckermannSteering plugin in the SDF.
-  -->
   <material name="silver">   <color rgba="1.0 0.4 0.0 1.0"/> </material>
-  <material name="dark">     <color rgba="0.10 0.10 0.10 1.0"/> </material>
   <material name="blue">     <color rgba="0.40 0.60 0.90 0.7"/> </material>
   <material name="red">      <color rgba="0.80 0.10 0.10 1.0"/> </material>
-  <!-- base_footprint (Nav2 convention) -->
-  <link name="base_footprint"/>
-  <joint name="base_footprint_joint" type="fixed">
-    <parent link="base_footprint"/>
-    <child  link="base_link"/>
-    <origin xyz="0 0 0.1" rpy="0 0 0"/>
-  </joint>
-  <!-- base_link — main body -->
+  <material name="dark">     <color rgba="0.10 0.10 0.10 1.0"/> </material>
   <link name="base_link">
-    <inertial>
-      <mass value="800.0"/>
-      <origin xyz="0 0 0.125"/>
-      <inertia ixx="200" iyy="800" izz="900" ixy="0" ixz="0" iyz="0"/>
-    </inertial>
     <visual>
-      <origin xyz="0 0 0.125"/>
       <geometry><box size="0.8 0.4 0.25"/></geometry>
       <material name="silver"/>
     </visual>
     <visual>
-      <origin xyz="-0.3 0 1.05"/>
-      <geometry><box size="0.4 0.32 0.18"/></geometry>
+      <origin xyz="-0.05 0 0.2"/>
+      <geometry><box size="0.35 0.3 0.15"/></geometry>
       <material name="blue"/>
     </visual>
     <collision>
-      <origin xyz="0 0 0.125"/>
       <geometry><box size="0.8 0.4 0.25"/></geometry>
     </collision>
   </link>
-  <!-- Front-left steering pivot -->
-  <link name="fl_steering_link">
-    <inertial><mass value="0.1"/>
-      <inertia ixx="0.001" iyy="0.001" izz="0.001" ixy="0" ixz="0" iyz="0"/>
-    </inertial>
+  <link name="left_wheel">
+    <visual><origin rpy="1.5708 0 0"/><geometry><cylinder radius="0.15" length="0.06"/></geometry><material name="dark"/></visual>
   </link>
-  <joint name="fl_steer_j" type="revolute">
-    <parent link="base_link"/> <child link="fl_steering_link"/>
-    <origin xyz="0.3 0.22 0"/>
-    <axis xyz="0 0 1"/>
-    <limit lower="-0.6" upper="0.6" effort="100" velocity="1.0"/>
+  <joint name="left_wheel_joint" type="continuous">
+    <parent link="base_link"/> <child link="left_wheel"/>
+    <origin xyz="0 0.22 0"/> <axis xyz="0 1 0"/>
   </joint>
-  <!-- Front-right steering pivot -->
-  <link name="fr_steering_link">
-    <inertial><mass value="0.1"/>
-      <inertia ixx="0.001" iyy="0.001" izz="0.001" ixy="0" ixz="0" iyz="0"/>
-    </inertial>
+  <link name="right_wheel">
+    <visual><origin rpy="1.5708 0 0"/><geometry><cylinder radius="0.15" length="0.06"/></geometry><material name="dark"/></visual>
   </link>
-  <joint name="fr_steer_j" type="revolute">
-    <parent link="base_link"/> <child link="fr_steering_link"/>
-    <origin xyz="0.3 -0.22 0"/>
-    <axis xyz="0 0 1"/>
-    <limit lower="-0.6" upper="0.6" effort="100" velocity="1.0"/>
+  <joint name="right_wheel_joint" type="continuous">
+    <parent link="base_link"/> <child link="right_wheel"/>
+    <origin xyz="0 -0.22 0"/> <axis xyz="0 1 0"/>
   </joint>
-  <!-- Front-left wheel -->
-  <link name="fl_wheel">
-    <inertial><mass value="15.0"/>
-      <inertia ixx="0.4" iyy="0.7" izz="0.4" ixy="0" ixz="0" iyz="0"/>
-    </inertial>
-    <visual>  <origin rpy="1.5708 0 0"/> <geometry><cylinder radius="0.1" length="0.06"/></geometry> <material name="dark"/> </visual>
-    <collision><origin rpy="1.5708 0 0"/> <geometry><cylinder radius="0.1" length="0.06"/></geometry></collision>
+  <link name="caster">
+    <visual><geometry><sphere radius="0.08"/></geometry><material name="dark"/></visual>
   </link>
-  <joint name="fl_j" type="revolute">
-    <parent link="fl_steering_link"/> <child link="fl_wheel"/>
-    <axis xyz="0 1 0"/>
-    <limit lower="-1e10" upper="1e10" effort="1000" velocity="10"/>
+  <joint name="caster_joint" type="fixed">
+    <parent link="base_link"/> <child link="caster"/>
+    <origin xyz="0.35 0 -0.05"/>
   </joint>
-  <!-- Front-right wheel -->
-  <link name="fr_wheel">
-    <inertial><mass value="15.0"/>
-      <inertia ixx="0.4" iyy="0.7" izz="0.4" ixy="0" ixz="0" iyz="0"/>
-    </inertial>
-    <visual>  <origin rpy="1.5708 0 0"/> <geometry><cylinder radius="0.1" length="0.06"/></geometry> <material name="dark"/> </visual>
-    <collision><origin rpy="1.5708 0 0"/> <geometry><cylinder radius="0.1" length="0.06"/></geometry></collision>
-  </link>
-  <joint name="fr_j" type="revolute">
-    <parent link="fr_steering_link"/> <child link="fr_wheel"/>
-    <axis xyz="0 1 0"/>
-    <limit lower="-1e10" upper="1e10" effort="1000" velocity="10"/>
-  </joint>
-  <!-- Rear-left wheel -->
-  <link name="rl_wheel">
-    <inertial><mass value="15.0"/>
-      <inertia ixx="0.4" iyy="0.7" izz="0.4" ixy="0" ixz="0" iyz="0"/>
-    </inertial>
-    <visual>  <origin rpy="1.5708 0 0"/> <geometry><cylinder radius="0.1" length="0.06"/></geometry> <material name="dark"/> </visual>
-    <collision><origin rpy="1.5708 0 0"/> <geometry><cylinder radius="0.1" length="0.06"/></geometry></collision>
-  </link>
-  <joint name="rl_j" type="revolute">
-    <parent link="base_link"/> <child link="rl_wheel"/>
-    <origin xyz="-0.3 0.22 0"/>
-    <axis xyz="0 1 0"/>
-    <limit lower="-1e10" upper="1e10" effort="1000" velocity="10"/>
-  </joint>
-  <!-- Rear-right wheel -->
-  <link name="rr_wheel">
-    <inertial><mass value="15.0"/>
-      <inertia ixx="0.4" iyy="0.7" izz="0.4" ixy="0" ixz="0" iyz="0"/>
-    </inertial>
-    <visual>  <origin rpy="1.5708 0 0"/> <geometry><cylinder radius="0.1" length="0.06"/></geometry> <material name="dark"/> </visual>
-    <collision><origin rpy="1.5708 0 0"/> <geometry><cylinder radius="0.1" length="0.06"/></geometry></collision>
-  </link>
-  <joint name="rr_j" type="revolute">
-    <parent link="base_link"/> <child link="rr_wheel"/>
-    <origin xyz="-0.3 -0.22 0"/>
-    <axis xyz="0 1 0"/>
-    <limit lower="-1e10" upper="1e10" effort="1000" velocity="10"/>
-  </joint>
-  <!-- LiDAR link (z=1.5m above base_link) -->
   <link name="lidar_link">
-    <inertial><mass value="0.5"/>
-      <inertia ixx="0.001" iyy="0.001" izz="0.001" ixy="0" ixz="0" iyz="0"/>
-    </inertial>
     <visual><geometry><cylinder radius="0.08" length="0.12"/></geometry><material name="red"/></visual>
-    <collision><geometry><cylinder radius="0.08" length="0.12"/></geometry></collision>
   </link>
   <joint name="lidar_joint" type="fixed">
     <parent link="base_link"/> <child link="lidar_link"/>
-    <origin xyz="0 0 0.45"/>
+    <origin xyz="0 0 0.3"/>
   </joint>
-  <!-- IMU link (at base_link origin) -->
-  <link name="imu_link">
-    <inertial><mass value="0.01"/>
-      <inertia ixx="0.0001" iyy="0.0001" izz="0.0001" ixy="0" ixz="0" iyz="0"/>
-    </inertial>
-  </link>
+  <link name="imu_link"/>
   <joint name="imu_joint" type="fixed">
     <parent link="base_link"/> <child link="imu_link"/>
